Commit message: gfdvxfdvsdx

File: body.urdf (robot description, URDF)
Before this commit: robot robot, 3 links, 2 joints
Joints:
- joint Torso BackLeg: origin xyz=-1 0 0.5 rpy=0 0 0 -> xyz=-0.5 0 1 rpy=0 0 0
- joint Torso FrontLeg: origin xyz=1 0 0.5 rpy=0 0 0 -> xyz=0.5 0 1 rpy=0 0 0

Commit message: testing new creatures

File: body.urdf (robot description, URDF)
Before this commit: robot robot, 3 links, 2 joints
Links:
- removed link BackLeg
- removed link FrontLeg
- added link BLL, mass 1; collision box size=0.1 0.1 0.5; visual box size=0.1 0.1 0.5
- added link BLT, mass 1; collision box size=0.15 0.15 0.5; visual box size=0.15 0.15 0.5
- added link BRL, mass 1; collision box size=0.1 0.1 0.5; visual box size=0.1 0.1 0.5
- added link BRT, mass 1; collision box size=0.15 0.15 0.5; visual box size=0.15 0.15 0.5
- added link FLL, mass 1; collision box size=0.1 0.1 0.5; visual box size=0.1 0.1 0.5
- added link FLT, mass 1; collision box size=0.15 0.15 0.75; visual box size=0.15 0.15 0.75
- added link FRL, mass 1; collision box size=0.1 0.1 0.5; visual box size=0.1 0.1 0.5
- added link FRT, mass 1; collision box size=0.15 0.15 0.75; visual box size=0.15 0.15 0.75
- link Torso: geometry collision box size=1 0.5 0.5; visual box size=1 0.5 0.5
Joints:
- removed joint Torso BackLeg
- removed joint Torso FrontLeg
- added joint BLT_BLL: type revolute, parent BLT, child BLL, origin xyz=0 0 -0.5 rpy=0 0 0, axis 0 1 0, limit lower=-3.14159 upper=3.14159 effort=0.0 velocity=0.0
- added joint BRT_BRL: type revolute, parent BRT, child BRL, origin xyz=0 0 -0.5 rpy=0 0 0, axis 0 1 0, limit lower=-3.14159 upper=3.14159 effort=0.0 velocity=0.0
- added joint FLT_FLL: type revolute, parent FLT, child FLL, origin xyz=0 0 -0.5 rpy=0 0 0, axis 0 1 0, limit lower=-3.14159 upper=3.14159 effort=0.0 velocity=0.0
- added joint FRT_FRL: type revolute, parent FRT, child FRL, origin xyz=0 0 -0.5 rpy=0 0 0, axis 0 1 0, limit lower=-3.14159 upper=3.14159 effort=0.0 velocity=0.0
- added joint Torso_BLT: type revolute, parent Torso, child BLT, origin xyz=.425 0.1775 1 rpy=0 0 0, axis 0 1 0, limit lower=-3.14159 upper=3.14159 effort=0.0 velocity=0.0
- added joint Torso_BRT: type revolute, parent Torso, child BRT, origin xyz=.425 -0.1775 1 rpy=0 0 0, axis 0 1 0, limit lower=-3.14159 upper=3.14159 effort=0.0 velocity=0.0
- added joint Torso_FLT: type revolute, parent Torso, child FLT, origin xyz=-.425 0.1775 0.875 rpy=0 0 0, axis 0 1 0, limit lower=-3.14159 upper=3.14159 effort=0.0 velocity=0.0
- added joint Torso_FRT: type revolute, parent Torso, child FRT, origin xyz=-.425 -0.1775 0.875 rpy=0 0 0, axis 0 1 0, limit lower=-3.14159 upper=3.14159 effort=0.0 velocity=0.0
